Commit message: creating the leo tank platform

File: description/gazebo_control.xacro (robot description, xacro)
@@ -6,5 +6,5 @@
             <left_joint>left_wheel_joint</left_joint>
             <right_joint>right_wheel_joint</right_joint>
-            <wheel_separation>0.22</wheel_separation>
+            <wheel_separation>0.17</wheel_separation>
             <wheel_diameter>0.07</wheel_diameter>
             <!-- LIMITS       -->

File: description/pulsepusher.xacro (robot description, xacro)
@@ -103,11 +103,16 @@
     <gazebo reference="left_wheel">
         <material>Gazebo/Blue</material>
-    </gazebo>
-    <joint name="left_wheel_joint_f" type="continuous">
+        <mu1 value="100000000000000.0" /><!-- 0.001-->
+        <mu2 value="100000000000000.0" />
+        <kp value="1000000000000.0" />
+        <kd value="10"/>
+        <minDepth>0.001</minDepth>
+        <maxVel>0.1</maxVel>
+        <fdir1>1 0 0</fdir1>
+    </gazebo>
+    <joint name="left_wheel_joint_f" type="fixed">
         <origin xyz="0.15 0.085 0.0" rpy="-${pi/2} 0.0 0.0" />
         <parent link="base_link" />
         <child link="left_wheel_f" />
-        <axis xyz="0.0 0.0 1.0" />
-        <limit lower="0.0" upper="0.0" effort="0.0" velocity="0.0" />
     </joint>
     <link name="left_wheel_f">
@@ -129,11 +134,16 @@
     <gazebo reference="left_wheel_f">
         <material>Gazebo/Blue</material>
-    </gazebo>
-    <joint name="left_wheel_joint_r" type="continuous">
+        <mu1 value="0.1" /><!-- 0.001-->
+        <mu2 value="0.1" />
+        <kp value="1000000.0" />
+        <kd value="10"/>
+        <minDepth>0.001</minDepth>
+        <maxVel>0.1</maxVel>
+        <fdir1>1 0 0</fdir1>
+    </gazebo>
+    <joint name="left_wheel_joint_r" type="fixed">
         <origin xyz="-0.15 0.085 0.0" rpy="-${pi/2} 0.0 0.0" />
         <parent link="base_link" />
         <child link="left_wheel_r" />
-        <axis xyz="0.0 0.0 1.0" />
-        <limit lower="0.0" upper="0.0" effort="0.0" velocity="0.0" />
     </joint>
     <link name="left_wheel_r">
@@ -155,4 +165,11 @@
     <gazebo reference="left_wheel_r">
         <material>Gazebo/Blue</material>
+        <mu1 value="0.1" /><!-- 0.001-->
+        <mu2 value="0.1" />
+        <kp value="1000000.0" />
+        <kd value="10"/>
+        <minDepth>0.001</minDepth>
+        <maxVel>0.1</maxVel>
+        <fdir1>1 0 0</fdir1>
     </gazebo>
     <!-- RIGHT WHEEL LINK -->
@@ -182,11 +199,16 @@
     <gazebo reference="right_wheel">
         <material>Gazebo/Blue</material>
-    </gazebo>
-    <joint name="right_wheel_joint_f" type="continuous">
+        <mu1 value="100000000000000.0" /><!-- 0.001-->
+        <mu2 value="100000000000000.0" />
+        <kp value="1000000000000.0" />
+        <kd value="10"/>
+        <minDepth>0.001</minDepth>
+        <maxVel>0.1</maxVel>
+        <fdir1>1 0 0</fdir1>
+    </gazebo>
+    <joint name="right_wheel_joint_f" type="fixed">
         <origin xyz="0.15 -0.085 0.0" rpy="${pi/2} 0.0 0.0" />
         <parent link="base_link" />
         <child link="right_wheel_f" />
-        <axis xyz="0.0 0.0 -1.0" />
-        <limit lower="0.0" upper="0.0" effort="0.0" velocity="0.0" />
     </joint>
     <link name="right_wheel_f">
@@ -208,11 +230,16 @@
     <gazebo reference="right_wheel_f">
         <material>Gazebo/Blue</material>
-    </gazebo>
-    <joint name="right_wheel_joint_r" type="continuous">
+        <mu1 value="0.1" /><!-- 0.001-->
+        <mu2 value="0.1" />
+        <kp value="1000000.0" />
+        <kd value="10"/>
+        <minDepth>0.001</minDepth>
+        <maxVel>0.1</maxVel>
+        <fdir1>1 0 0</fdir1>
+    </gazebo>
+    <joint name="right_wheel_joint_r" type="fixed">
         <origin xyz="-0.15 -0.085 0.0" rpy="${pi/2} 0.0 0.0" />
         <parent link="base_link" />
         <child link="right_wheel_r" />
-        <axis xyz="0.0 0.0 -1.0" />
-        <limit lower="0.0" upper="0.0" effort="0.0" velocity="0.0" />
     </joint>
     <link name="right_wheel_r">
@@ -234,4 +261,11 @@
     <gazebo reference="right_wheel_r">
         <material>Gazebo/Blue</material>
+        <mu1 value="0.1" /><!-- 0.001-->
+        <mu2 value="0.1" />
+        <kp value="1000000.0" />
+        <kd value="10"/>
+        <minDepth>0.001</minDepth>
+        <maxVel>0.1</maxVel>
+        <fdir1>1 0 0</fdir1>
     </gazebo>
 </robot>

File: description/robot.urdf.xacro (robot description, xacro)
@@ -2,4 +2,5 @@
 <robot xmlns:xacro="http://www.ros.org/wiki/xacro"  name="pulsepusher">
     <xacro:include filename="pulsepusher.xacro" />
+    <xacro:include filename="gazebo_control.xacro"/>
    <!-- <xacro:include filename="lidar.xacro" />
     <xacro:include filename="camera.xacro" />
