Commit message: pulsepusher von homerobot zu leotank ueberarbeiten

File: description/pulsepusher.xacro (robot description, xacro)
@@ -28,11 +28,11 @@
         <parent link="base_link"/>
         <child link="chassis"/>
-        <origin xyz="-0.093 0.0 0.0"/>
+        <origin xyz="0.0 0.0 0.0"/>
     </joint>
     <link name="chassis">
         <visual>
-            <origin xyz="0.093 0.0 0.02"/>
+            <origin xyz="0 0 0.0"/>
             <geometry>
-                <cylinder radius="0.093" length="0.045"/>
+                <box size="0.47 0.13 0.1"/>
             </geometry>
             <material name="orange"/>
@@ -41,13 +41,13 @@
             <origin xyz="0.093 0.0 0.075"/>
             <geometry>
-                <cylinder radius="0.093" length="0.045"/>
+                <box size="0.47 0.13 0.1"/>
             </geometry>
         </collision>
-        <xacro:inertial_cylinder mass="0.5" length="0.045" radius="0.093">
-            <origin xyz="0.0 0.0 0.0" rpy="0.0 0.0 0.0"/>
-        </xacro:inertial_cylinder>
+        <xacro:inertial_box mass="0.3" x="0.47" y="0.12" z="0.1">
+            <origion xyz="0.0 0.0 0.0" rpy="0.0 0.0 0.0"/>
+        </xacro:inertial_box>
     </link>
     <gazebo reference="chassis">
-        <material>Gazebo/Orange</material>
+        <material>Gazebo/Black</material>
     </gazebo>
         <!-- LEFT WHEEL LINK -->
@@ -159,5 +159,5 @@
         <mu2 value="0.001"/>
     </gazebo>
-    <!-- Body Part -->
+    <!-- Body Part
     <link name="body">
         <visual>
@@ -183,53 +183,4 @@
         <child link="body"/>
         <origin xyz="0.0 0.0 0.21"/>
-    </joint>
-    <!-- LCD DISPLAY and In_display  -->
-    <link name="display">
-        <visual>
-            <geometry>
-                <box size="0.09 0.09 0.05"/>
-            </geometry>
-            <material name="black"/>
-        </visual>
-        <collision>
-            <geometry>
-                <box size="0.09 0.09 0.03"/>
-            </geometry>
-        </collision>
-        <xacro:inertial_box mass="0.1" x="0.09" y="0.09" z="0.05">
-            <origion xyz="0.0 0.0 0.0" rpy="0.0 0.0 0.0"/>
-        </xacro:inertial_box>
-    </link>
-    <gazebo reference="display">
-        <material>Gazebo/Black</material>
-    </gazebo>
-    <joint name="display_body_joint" type="fixed">
-        <origin xyz="0.08 0.0 0.11" rpy="0 0.0 0.0"/>
-        <parent link="body"/>
-        <child link="display"/>
-    </joint>
-    <link name="in_display">
-        <visual>
-            <geometry>
-                <box size="0.09 0.07 0.03"/>
-            </geometry>
-            <material name="green"/>
-        </visual>
-        <collision>
-            <geometry>
-                <box size="0.09 0.07 0.03"/>
-            </geometry>
-        </collision>
-        <xacro:inertial_box mass="0.1" x="0.09" y="0.09" z="0.03">
-            <origion xyz="0.0 0.0 0.0" rpy="0.0 0.0 0.0"/>
-        </xacro:inertial_box>
-    </link>
-    <gazebo reference="in_display">
-        <material>Gazebo/Green</material>
-    </gazebo>
-    <joint name="in_display_body_joint" type="fixed">
-        <origin xyz="0.085 0.0 0.11" rpy="0 0.0 0.0"/>
-        <parent link="body"/>
-        <child link="in_display"/>
-    </joint>
+    </joint>-->
 </robot>

File: description/robot.urdf.xacro (robot description, xacro)
@@ -2,8 +2,7 @@
 <robot xmlns:xacro="http://www.ros.org/wiki/xacro"  name="pulsepusher">
     <xacro:include filename="pulsepusher.xacro" />
-    <xacro:include filename="lidar.xacro" />
+   <!-- <xacro:include filename="lidar.xacro" />
     <xacro:include filename="camera.xacro" />
-    <!-- <xacro:include filename="ros2_control.xacro" /> -->
-    <xacro:include filename="gazebo_control.xacro"/>
+     <xacro:include filename="ros2_control.xacro" /> -->
 <!--
     <xacro:if value="$(arg use_ros2_control)">

Commit message: test an urdf

File: description/pulsepusher.xacro (robot description, xacro)
@@ -32,5 +32,5 @@
     <link name="chassis">
         <visual>
-            <origin xyz="0 0 0.0"/>
+            <origin xyz="0 0 0.05"/>
             <geometry>
                 <box size="0.47 0.13 0.1"/>
@@ -51,8 +51,8 @@
         <material>Gazebo/Black</material>
     </gazebo>
-        <!-- LEFT WHEEL LINK -->
+        <!-- LEFT WHEEL LINK  Section-->
     <joint name="left_wheel_joint" type="continuous">
-        <origin xyz="0.0 0.11 0.0" rpy="-${pi/2} 0.0 0.0"/>
-        <parent link="base_link"/>
+        <origin xyz="0.0 0.09 -0.025" rpy="-${pi/2} 0.0 0.0"/>
+        <parent link="chassis"/>
         <child link="left_wheel"/>
         <axis xyz="0.0 0.0 1.0"/>
@@ -78,8 +78,60 @@
         <material>Gazebo/Blue</material>
     </gazebo>
+    <joint name="left_wheel_joint_f" type="continuous">
+        <origin xyz="0.15 0.09 -0.025" rpy="-${pi/2} 0.0 0.0"/>
+        <parent link="chassis"/>
+        <child link="left_wheel_f"/>
+        <axis xyz="0.0 0.0 1.0"/>
+        <limit lower="0.0" upper="0.0" effort="0.0" velocity="0.0"/>
+    </joint>
+    <link name="left_wheel_f">
+        <visual>
+            <geometry>
+                <cylinder radius="0.035" length="0.028"/>
+            </geometry>
+            <material name="blue"/>
+        </visual>
+        <collision>
+            <geometry>
+                <cylinder radius="0.035" length="0.028"/>
+            </geometry>
+        </collision>
+        <xacro:inertial_cylinder mass="0.1" length="0.028" radius="0.035">
+            <origin xyz="0.0 0.0 0.0" rpy="0.0 0.0 0.0"/>
+        </xacro:inertial_cylinder>
+    </link>
+    <gazebo reference="left_wheel_f">
+        <material>Gazebo/Blue</material>
+    </gazebo>
+    <joint name="left_wheel_joint_r" type="continuous">
+        <origin xyz="-0.15 0.09 -0.025" rpy="-${pi/2} 0.0 0.0"/>
+        <parent link="chassis"/>
+        <child link="left_wheel_r"/>
+        <axis xyz="0.0 0.0 1.0"/>
+        <limit lower="0.0" upper="0.0" effort="0.0" velocity="0.0"/>
+    </joint>
+    <link name="left_wheel_r">
+        <visual>
+            <geometry>
+                <cylinder radius="0.035" length="0.028"/>
+            </geometry>
+            <material name="blue"/>
+        </visual>
+        <collision>
+            <geometry>
+                <cylinder radius="0.035" length="0.028"/>
+            </geometry>
+        </collision>
+        <xacro:inertial_cylinder mass="0.1" length="0.028" radius="0.035">
+            <origin xyz="0.0 0.0 0.0" rpy="0.0 0.0 0.0"/>
+        </xacro:inertial_cylinder>
+    </link>
+    <gazebo reference="left_wheel_r">
+        <material>Gazebo/Blue</material>
+    </gazebo>
     <!-- RIGHT WHEEL LINK -->
     <joint name="right_wheel_joint" type="continuous">
-        <origin xyz="0.0 -0.11 0.0" rpy="${pi/2} 0.0 0.0"/>
-        <parent link="base_link"/>
+        <origin xyz="0.0 -0.09 -0.025" rpy="${pi/2} 0.0 0.0"/>
+        <parent link="chassis"/>
         <child link="right_wheel"/>
         <axis xyz="0.0 0.0 -1.0"/>
@@ -105,5 +157,57 @@
         <material>Gazebo/Blue</material>
     </gazebo>
-    <!-- CASTER WHEEL FRONT LINK -->
+    <joint name="right_wheel_joint_f" type="continuous">
+        <origin xyz="0.15 -0.09 -0.025" rpy="${pi/2} 0.0 0.0"/>
+        <parent link="chassis"/>
+        <child link="right_wheel_f"/>
+        <axis xyz="0.0 0.0 -1.0"/>
+        <limit lower="0.0" upper="0.0" effort="0.0" velocity="0.0"/>
+    </joint>
+    <link name="right_wheel_f">
+        <visual>
+            <geometry>
+                <cylinder radius="0.035" length="0.028"/>
+            </geometry>
+            <material name="blue"/>
+        </visual>
+        <collision>
+            <geometry>
+                <cylinder radius="0.035" length="0.028"/>
+            </geometry>
+        </collision>
+        <xacro:inertial_cylinder mass="0.1" length="0.028" radius="0.035">
+            <origin xyz="0.0 0.0 0.0" rpy="0.0 0.0 0.0"/>
+        </xacro:inertial_cylinder>
+    </link>
+    <gazebo reference="right_wheel_f">
+        <material>Gazebo/Blue</material>
+    </gazebo>
+    <joint name="right_wheel_joint_r" type="continuous">
+        <origin xyz="-0.15 -0.09 -0.025" rpy="${pi/2} 0.0 0.0"/>
+        <parent link="chassis"/>
+        <child link="right_wheel_r"/>
+        <axis xyz="0.0 0.0 -1.0"/>
+        <limit lower="0.0" upper="0.0" effort="0.0" velocity="0.0"/>
+    </joint>
+    <link name="right_wheel_r">
+        <visual>
+            <geometry>
+                <cylinder radius="0.035" length="0.028"/>
+            </geometry>
+            <material name="blue"/>
+        </visual>
+        <collision>
+            <geometry>
+                <cylinder radius="0.035" length="0.028"/>
+            </geometry>
+        </collision>
+        <xacro:inertial_cylinder mass="0.1" length="0.028" radius="0.035">
+            <origin xyz="0.0 0.0 0.0" rpy="0.0 0.0 0.0"/>
+        </xacro:inertial_cylinder>
+    </link>
+    <gazebo reference="right_wheel_r">
+        <material>Gazebo/Blue</material>
+    </gazebo>
+    <!-- CASTER WHEEL FRONT LINK
     <joint name="caster_wheel_front_joint" type="fixed">
         <parent link="base_link"/>
@@ -131,6 +235,6 @@
         <mu1 value="0.001"/>
         <mu2 value="0.001"/>
-    </gazebo>
-    <!-- CASTER WHEEL REAR LINK -->
+    </gazebo> -->
+    <!-- CASTER WHEEL REAR LINK
     <joint name="caster_wheel_rear_joint" type="fixed">
         <parent link="base_link"/>
@@ -158,5 +262,5 @@
         <mu1 value="0.001"/>
         <mu2 value="0.001"/>
-    </gazebo>
+    </gazebo> -->
     <!-- Body Part
     <link name="body">
