Commit message: tank ground

File: description/pulsepusher.xacro (robot description, xacro)
@@ -1,23 +1,23 @@
 <?xml version="1.0"?>
-<robot xmlns:xacro="http://www.ros.org/wiki/xacro" >
-        <xacro:include filename="inertial_macros.xacro"/>
-            <!-- Farben -->
+<robot xmlns:xacro="http://www.ros.org/wiki/xacro">
+    <xacro:include filename="inertial_macros.xacro" />
+    <!-- Farben -->
     <material name="white">
-        <color rgba="1 1 1 1"/>
+        <color rgba="1 1 1 1" />
     </material>
     <material name="black">
-        <color rgba="0 0 0 1"/>
+        <color rgba="0 0 0 1" />
     </material>
     <material name="blue">
-        <color rgba="0.2 0.2 1 1"/>
+        <color rgba="0.2 0.2 1 1" />
     </material>
     <material name="yellow">
-        <color rgba="1 1 0 1"/>
+        <color rgba="1 1 0 1" />
     </material>
     <material name="orange">
-        <color rgba="1 0.3 0.1 1"/>
+        <color rgba="1 0.3 0.1 1" />
     </material>
     <material name="green">
-        <color rgba="0.0 1.0 0.0 1.0"/>
+        <color rgba="0.0 1.0 0.0 1.0" />
     </material>
     <!-- BASE LINK -->
@@ -26,24 +26,24 @@
     <!-- CHASSIS LINK -->
     <joint name="cassis_joint" type="fixed">
-        <parent link="base_link"/>
-        <child link="chassis"/>
-        <origin xyz="0.0 0.0 0.0"/>
+        <parent link="base_link" />
+        <child link="chassis" />
+        <origin xyz="-0.25 0.0 0.0" />
     </joint>
     <link name="chassis">
         <visual>
-            <origin xyz="0 0 0.05"/>
-            <geometry>
-                <box size="0.47 0.13 0.1"/>
-            </geometry>
-            <material name="orange"/>
-        </visual>
-        <collision>
-            <origin xyz="0.093 0.0 0.075"/>
-            <geometry>
-                <box size="0.47 0.13 0.1"/>
-            </geometry>
-        </collision>
-        <xacro:inertial_box mass="0.3" x="0.47" y="0.12" z="0.1">
-            <origion xyz="0.0 0.0 0.0" rpy="0.0 0.0 0.0"/>
+            <origin xyz="0.25 0.0 0.03" />
+            <geometry>
+                <box size="0.5 0.13 0.06" />
+            </geometry>
+            <material name="black" />
+        </visual>
+        <collision>
+            <origin xyz="0.25 0.0 0.03" />
+            <geometry>
+                <box size="0.5 0.13 0.06" />
+            </geometry>
+        </collision>
+        <xacro:inertial_box mass="0.3" x="0.5" y="0.13" z="0.06">
+            <origion xyz="0.0 0.0 0.0" rpy="0.0 0.0 0.0" />
         </xacro:inertial_box>
     </link>
@@ -51,26 +51,52 @@
         <material>Gazebo/Black</material>
     </gazebo>
-        <!-- LEFT WHEEL LINK  Section-->
+    <joint name="cassis_top_joint" type="fixed">
+        <parent link="chassis" />
+        <child link="chassis_top" />
+        <origin xyz="0.0 0.0 0.0" />
+    </joint>
+    <link name="chassis_top">
+        <visual>
+            <origin xyz="0.25 0 0.06" />
+            <geometry>
+                <box size="0.5 0.22 0.02" />
+            </geometry>
+            <material name="black" />
+        </visual>
+        <collision>
+            <origin xyz="0.25 0 0.06" />
+            <geometry>
+                <box size="0.5 0.22 0.02" />
+            </geometry>
+        </collision>
+        <xacro:inertial_box mass="0.1" x="0.5" y="0.22" z="0.02">
+            <origion xyz="0.0 0.0 0.0" rpy="0.0 0.0 0.0" />
+        </xacro:inertial_box>
+    </link>
+    <gazebo reference="chassis_top">
+        <material>Gazebo/Black</material>
+    </gazebo>
+    <!-- LEFT WHEEL LINK  Section-->
     <joint name="left_wheel_joint" type="continuous">
-        <origin xyz="0.0 0.09 -0.025" rpy="-${pi/2} 0.0 0.0"/>
-        <parent link="chassis"/>
-        <child link="left_wheel"/>
-        <axis xyz="0.0 0.0 1.0"/>
-        <limit lower="0.0" upper="0.0" effort="0.0" velocity="0.0"/>
+        <origin xyz="0.0 0.085 0.0" rpy="-${pi/2} 0.0 0.0" />
+        <parent link="base_link" />
+        <child link="left_wheel" />
+        <axis xyz="0.0 0.0 1.0" />
+        <limit lower="0.0" upper="0.0" effort="0.0" velocity="0.0" />
     </joint>
     <link name="left_wheel">
         <visual>
             <geometry>
-                <cylinder radius="0.035" length="0.028"/>
-            </geometry>
-            <material name="blue"/>
-        </visual>
-        <collision>
-            <geometry>
-                <cylinder radius="0.035" length="0.028"/>
-            </geometry>
-        </collision>
-        <xacro:inertial_cylinder mass="0.1" length="0.028" radius="0.035">
-            <origin xyz="0.0 0.0 0.0" rpy="0.0 0.0 0.0"/>
+                <cylinder radius="0.035" length="0.028" />
+            </geometry>
+            <material name="blue" />
+        </visual>
+        <collision>
+            <geometry>
+                <sphere radius="0.035" />
+            </geometry>
+        </collision>
+        <xacro:inertial_cylinder mass="0.1" length="0.028" radius="0.035">
+            <origin xyz="0.0 0.0 0.0" rpy="0.0 0.0 0.0" />
         </xacro:inertial_cylinder>
     </link>
@@ -79,24 +105,24 @@
     </gazebo>
     <joint name="left_wheel_joint_f" type="continuous">
-        <origin xyz="0.15 0.09 -0.025" rpy="-${pi/2} 0.0 0.0"/>
-        <parent link="chassis"/>
-        <child link="left_wheel_f"/>
-        <axis xyz="0.0 0.0 1.0"/>
-        <limit lower="0.0" upper="0.0" effort="0.0" velocity="0.0"/>
+        <origin xyz="0.15 0.085 0.0" rpy="-${pi/2} 0.0 0.0" />
+        <parent link="base_link" />
+        <child link="left_wheel_f" />
+        <axis xyz="0.0 0.0 1.0" />
+        <limit lower="0.0" upper="0.0" effort="0.0" velocity="0.0" />
     </joint>
     <link name="left_wheel_f">
         <visual>
             <geometry>
-                <cylinder radius="0.035" length="0.028"/>
-            </geometry>
-            <material name="blue"/>
-        </visual>
-        <collision>
-            <geometry>
-                <cylinder radius="0.035" length="0.028"/>
-            </geometry>
-        </collision>
-        <xacro:inertial_cylinder mass="0.1" length="0.028" radius="0.035">
-            <origin xyz="0.0 0.0 0.0" rpy="0.0 0.0 0.0"/>
+                <cylinder radius="0.035" length="0.028" />
+            </geometry>
+            <material name="blue" />
+        </visual>
+        <collision>
+            <geometry>
+                <sphere radius="0.035" />
+            </geometry>
+        </collision>
+        <xacro:inertial_cylinder mass="0.1" length="0.028" radius="0.035">
+            <origin xyz="0.0 0.0 0.0" rpy="0.0 0.0 0.0" />
         </xacro:inertial_cylinder>
     </link>
@@ -105,24 +131,24 @@
     </gazebo>
     <joint name="left_wheel_joint_r" type="continuous">
-        <origin xyz="-0.15 0.09 -0.025" rpy="-${pi/2} 0.0 0.0"/>
-        <parent link="chassis"/>
-        <child link="left_wheel_r"/>
-        <axis xyz="0.0 0.0 1.0"/>
-        <limit lower="0.0" upper="0.0" effort="0.0" velocity="0.0"/>
+        <origin xyz="-0.15 0.085 0.0" rpy="-${pi/2} 0.0 0.0" />
+        <parent link="base_link" />
+        <child link="left_wheel_r" />
+        <axis xyz="0.0 0.0 1.0" />
+        <limit lower="0.0" upper="0.0" effort="0.0" velocity="0.0" />
     </joint>
     <link name="left_wheel_r">
         <visual>
             <geometry>
-                <cylinder radius="0.035" length="0.028"/>
-            </geometry>
-            <material name="blue"/>
-        </visual>
-        <collision>
-            <geometry>
-                <cylinder radius="0.035" length="0.028"/>
-            </geometry>
-        </collision>
-        <xacro:inertial_cylinder mass="0.1" length="0.028" radius="0.035">
-            <origin xyz="0.0 0.0 0.0" rpy="0.0 0.0 0.0"/>
+                <cylinder radius="0.035" length="0.028" />
+            </geometry>
+            <material name="blue" />
+        </visual>
+        <collision>
+            <geometry>
+                <sphere radius="0.035" />
+            </geometry>
+        </collision>
+        <xacro:inertial_cylinder mass="0.1" length="0.028" radius="0.035">
+            <origin xyz="0.0 0.0 0.0" rpy="0.0 0.0 0.0" />
         </xacro:inertial_cylinder>
     </link>
@@ -132,24 +158,24 @@
     <!-- RIGHT WHEEL LINK -->
     <joint name="right_wheel_joint" type="continuous">
-        <origin xyz="0.0 -0.09 -0.025" rpy="${pi/2} 0.0 0.0"/>
-        <parent link="chassis"/>
-        <child link="right_wheel"/>
-        <axis xyz="0.0 0.0 -1.0"/>
-        <limit lower="0.0" upper="0.0" effort="0.0" velocity="0.0"/>
+        <origin xyz="0.0 -0.085 0.0" rpy="${pi/2} 0.0 0.0" />
+        <parent link="base_link" />
+        <child link="right_wheel" />
+        <axis xyz="0.0 0.0 -1.0" />
+        <limit lower="0.0" upper="0.0" effort="0.0" velocity="0.0" />
     </joint>
     <link name="right_wheel">
         <visual>
             <geometry>
-                <cylinder radius="0.035" length="0.028"/>
-            </geometry>
-            <material name="blue"/>
-        </visual>
-        <collision>
-            <geometry>
-                <cylinder radius="0.035" length="0.028"/>
-            </geometry>
-        </collision>
-        <xacro:inertial_cylinder mass="0.1" length="0.028" radius="0.035">
-            <origin xyz="0.0 0.0 0.0" rpy="0.0 0.0 0.0"/>
+                <cylinder radius="0.035" length="0.028" />
+            </geometry>
+            <material name="blue" />
+        </visual>
+        <collision>
+            <geometry>
+                <sphere radius="0.035" />
+            </geometry>
+        </collision>
+        <xacro:inertial_cylinder mass="0.1" length="0.028" radius="0.035">
+            <origin xyz="0.0 0.0 0.0" rpy="0.0 0.0 0.0" />
         </xacro:inertial_cylinder>
     </link>
@@ -158,24 +184,24 @@
     </gazebo>
     <joint name="right_wheel_joint_f" type="continuous">
-        <origin xyz="0.15 -0.09 -0.025" rpy="${pi/2} 0.0 0.0"/>
-        <parent link="chassis"/>
-        <child link="right_wheel_f"/>
-        <axis xyz="0.0 0.0 -1.0"/>
-        <limit lower="0.0" upper="0.0" effort="0.0" velocity="0.0"/>
+        <origin xyz="0.15 -0.085 0.0" rpy="${pi/2} 0.0 0.0" />
+        <parent link="base_link" />
+        <child link="right_wheel_f" />
+        <axis xyz="0.0 0.0 -1.0" />
+        <limit lower="0.0" upper="0.0" effort="0.0" velocity="0.0" />
     </joint>
     <link name="right_wheel_f">
         <visual>
             <geometry>
-                <cylinder radius="0.035" length="0.028"/>
-            </geometry>
-            <material name="blue"/>
-        </visual>
-        <collision>
-            <geometry>
-                <cylinder radius="0.035" length="0.028"/>
-            </geometry>
-        </collision>
-        <xacro:inertial_cylinder mass="0.1" length="0.028" radius="0.035">
-            <origin xyz="0.0 0.0 0.0" rpy="0.0 0.0 0.0"/>
+                <cylinder radius="0.035" length="0.028" />
+            </geometry>
+            <material name="blue" />
+        </visual>
+        <collision>
+            <geometry>
+                <sphere radius="0.035" />
+            </geometry>
+        </collision>
+        <xacro:inertial_cylinder mass="0.1" length="0.028" radius="0.035">
+            <origin xyz="0.0 0.0 0.0" rpy="0.0 0.0 0.0" />
         </xacro:inertial_cylinder>
     </link>
@@ -184,24 +210,24 @@
     </gazebo>
     <joint name="right_wheel_joint_r" type="continuous">
-        <origin xyz="-0.15 -0.09 -0.025" rpy="${pi/2} 0.0 0.0"/>
-        <parent link="chassis"/>
-        <child link="right_wheel_r"/>
-        <axis xyz="0.0 0.0 -1.0"/>
-        <limit lower="0.0" upper="0.0" effort="0.0" velocity="0.0"/>
+        <origin xyz="-0.15 -0.085 0.0" rpy="${pi/2} 0.0 0.0" />
+        <parent link="base_link" />
+        <child link="right_wheel_r" />
+        <axis xyz="0.0 0.0 -1.0" />
+        <limit lower="0.0" upper="0.0" effort="0.0" velocity="0.0" />
     </joint>
     <link name="right_wheel_r">
         <visual>
             <geometry>
-                <cylinder radius="0.035" length="0.028"/>
-            </geometry>
-            <material name="blue"/>
-        </visual>
-        <collision>
-            <geometry>
-                <cylinder radius="0.035" length="0.028"/>
-            </geometry>
-        </collision>
-        <xacro:inertial_cylinder mass="0.1" length="0.028" radius="0.035">
-            <origin xyz="0.0 0.0 0.0" rpy="0.0 0.0 0.0"/>
+                <cylinder radius="0.035" length="0.028" />
+            </geometry>
+            <material name="blue" />
+        </visual>
+        <collision>
+            <geometry>
+                <sphere radius="0.035" />
+            </geometry>
+        </collision>
+        <xacro:inertial_cylinder mass="0.1" length="0.028" radius="0.035">
+            <origin xyz="0.0 0.0 0.0" rpy="0.0 0.0 0.0" />
         </xacro:inertial_cylinder>
     </link>
@@ -209,82 +235,3 @@
         <material>Gazebo/Blue</material>
     </gazebo>
-    <!-- CASTER WHEEL FRONT LINK
-    <joint name="caster_wheel_front_joint" type="fixed">
-        <parent link="base_link"/>
-        <child link="caster_wheel_front"/>
-        <origin xyz="0.085 0.0 -0.016"/>
-    </joint>
-    <link name="caster_wheel_front">
-        <visual>
-            <geometry>
-                <sphere radius="0.018"/>
-            </geometry>
-            <material name="black"/>
-        </visual>
-        <collision>
-            <geometry>
-                <sphere radius="0.018"/>
-            </geometry>
-        </collision>
-        <xacro:inertial_sphere mass="0.3" radius="0.018">
-            <origin xyz="0.0 0.0 0.0" rpy="0.0 0.0 0.0"/>
-        </xacro:inertial_sphere>
-    </link>
-    <gazebo reference="caster_wheel_front">
-        <material>Gazebo/Black</material>
-        <mu1 value="0.001"/>
-        <mu2 value="0.001"/>
-    </gazebo> -->
-    <!-- CASTER WHEEL REAR LINK
-    <joint name="caster_wheel_rear_joint" type="fixed">
-        <parent link="base_link"/>
-        <child link="caster_wheel_rear"/>
-        <origin xyz="-0.085 0.0 -0.0165"/>
-    </joint>
-    <link name="caster_wheel_rear">
-        <visual>
-            <geometry>
-                <sphere radius="0.018"/>
-            </geometry>
-            <material name="black"/>
-        </visual>
-        <collision>
-            <geometry>
-                <sphere radius="0.018"/>
-            </geometry>
-        </collision>
-        <xacro:inertial_sphere mass="0.3" radius="0.018">
-            <origin xyz="0.0 0.0 0.0" rpy="0.0 0.0 0.0"/>
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
Commit message: start on pi

File: description/pulsepusher.xacro (robot description, xacro)
@@ -2,4 +2,5 @@
 <robot xmlns:xacro="http://www.ros.org/wiki/xacro">
     <xacro:include filename="inertial_macros.xacro" />
+    <xacro:include filename="pulse_gazebo.xacro" />
     <!-- Farben -->
     <material name="white">
@@ -101,14 +102,4 @@
         </xacro:inertial_cylinder>
     </link>
-    <gazebo reference="left_wheel">
-        <material>Gazebo/Blue</material>
-        <mu1 value="100000000000000.0" /><!-- 0.001-->
-        <mu2 value="100000000000000.0" />
-        <kp value="1000000000000.0" />
-        <kd value="10"/>
-        <minDepth>0.001</minDepth>
-        <maxVel>0.1</maxVel>
-        <fdir1>1 0 0</fdir1>
-    </gazebo>
     <joint name="left_wheel_joint_f" type="fixed">
         <origin xyz="0.15 0.085 0.0" rpy="-${pi/2} 0.0 0.0" />
@@ -132,14 +123,4 @@
         </xacro:inertial_cylinder>
     </link>
-    <gazebo reference="left_wheel_f">
-        <material>Gazebo/Blue</material>
-        <mu1 value="0.1" /><!-- 0.001-->
-        <mu2 value="0.1" />
-        <kp value="1000000.0" />
-        <kd value="10"/>
-        <minDepth>0.001</minDepth>
-        <maxVel>0.1</maxVel>
-        <fdir1>1 0 0</fdir1>
-    </gazebo>
     <joint name="left_wheel_joint_r" type="fixed">
         <origin xyz="-0.15 0.085 0.0" rpy="-${pi/2} 0.0 0.0" />
@@ -163,14 +144,4 @@
         </xacro:inertial_cylinder>
     </link>
-    <gazebo reference="left_wheel_r">
-        <material>Gazebo/Blue</material>
-        <mu1 value="0.1" /><!-- 0.001-->
-        <mu2 value="0.1" />
-        <kp value="1000000.0" />
-        <kd value="10"/>
-        <minDepth>0.001</minDepth>
-        <maxVel>0.1</maxVel>
-        <fdir1>1 0 0</fdir1>
-    </gazebo>
     <!-- RIGHT WHEEL LINK -->
     <joint name="right_wheel_joint" type="continuous">
@@ -197,14 +168,4 @@
         </xacro:inertial_cylinder>
     </link>
-    <gazebo reference="right_wheel">
-        <material>Gazebo/Blue</material>
-        <mu1 value="100000000000000.0" /><!-- 0.001-->
-        <mu2 value="100000000000000.0" />
-        <kp value="1000000000000.0" />
-        <kd value="10"/>
-        <minDepth>0.001</minDepth>
-        <maxVel>0.1</maxVel>
-        <fdir1>1 0 0</fdir1>
-    </gazebo>
     <joint name="right_wheel_joint_f" type="fixed">
         <origin xyz="0.15 -0.085 0.0" rpy="${pi/2} 0.0 0.0" />
@@ -228,14 +189,4 @@
         </xacro:inertial_cylinder>
     </link>
-    <gazebo reference="right_wheel_f">
-        <material>Gazebo/Blue</material>
-        <mu1 value="0.1" /><!-- 0.001-->
-        <mu2 value="0.1" />
-        <kp value="1000000.0" />
-        <kd value="10"/>
-        <minDepth>0.001</minDepth>
-        <maxVel>0.1</maxVel>
-        <fdir1>1 0 0</fdir1>
-    </gazebo>
     <joint name="right_wheel_joint_r" type="fixed">
         <origin xyz="-0.15 -0.085 0.0" rpy="${pi/2} 0.0 0.0" />
@@ -259,13 +210,3 @@
         </xacro:inertial_cylinder>
     </link>
-    <gazebo reference="right_wheel_r">
-        <material>Gazebo/Blue</material>
-        <mu1 value="0.1" /><!-- 0.001-->
-        <mu2 value="0.1" />
-        <kp value="1000000.0" />
-        <kd value="10"/>
-        <minDepth>0.001</minDepth>
-        <maxVel>0.1</maxVel>
-        <fdir1>1 0 0</fdir1>
-    </gazebo>
 </robot>

File: description/robot.urdf.xacro (robot description, xacro)
@@ -3,5 +3,5 @@
     <xacro:include filename="pulsepusher.xacro" />
     <xacro:include filename="gazebo_control.xacro"/>
-   <!-- <xacro:include filename="lidar.xacro" />
+ <!--    <xacro:include filename="lidar.xacro" />
     <xacro:include filename="camera.xacro" />
      <xacro:include filename="ros2_control.xacro" /> -->
