Commit message: urdf is ready. go to hardware

File: description/camera.xacro (robot description, xacro)
@@ -36,5 +36,5 @@
     </gazebo>
     <joint name="cam_body_joint" type="fixed">
-        <origin xyz="0.1 0.0 0.06" rpy="${pi/2} 0.0 0.0"/>
+        <origin xyz="0.1 0.0 0.06" rpy="0.0 0.0 0.0"/>
         <parent link="body"/>
         <child link="cam"/>

File: description/robot.urdf.xacro (robot description, xacro)
@@ -4,3 +4,4 @@
     <xacro:include filename="lidar.xacro" />
     <xacro:include filename="camera.xacro" />
+    <xacro:include filename="gazebo_control.xacro"/>
 </robot>

Commit message: added tower and cam

File: description/camera.xacro (robot description, xacro)
@@ -21,5 +21,5 @@
         <visual>
             <geometry>
-                <cylinder radius="0.01" length="0.05"/>
+                <cylinder radius="0.01" length="0.02"/>
             </geometry>
             <material name="black"/>
@@ -27,7 +27,10 @@
         <collision>
             <geometry>
-                <cylinder radius="0.01" length="0.05"/>
+                <cylinder radius="0.01" length="0.02"/>
             </geometry>
         </collision>
+        <xacro:inertial_cylinder mass="0.01" length="0.02" radius="0.01">
+            <origin xyz="0.0 0.0 0.0" rpy="0.0 0.0 0.0" />
+        </xacro:inertial_cylinder>
     </link>
     <link name="camera_link_optical"></link>
@@ -36,10 +39,10 @@
     </gazebo>
     <joint name="cam_body_joint" type="fixed">
-        <origin xyz="0.1 0.0 0.06" rpy="0.0 0.0 0.0"/>
-        <parent link="body"/>
+        <origin xyz="0.0 0.0 0.04" rpy="0.0 0.0 0.0"/>
+        <parent link="turm_top_r"/>
         <child link="cam"/>
     </joint>
     <joint name="linse_to_cam" type="fixed">
-        <origin xyz="0.0 0.0 0.0" rpy="0 ${pi/2} 0.0"/>
+        <origin xyz="0.015 0.0 0.0" rpy="0 ${pi/2} 0.0"/>
         <parent link="cam"/>
         <child link="cam_linse"/>

File: description/pulsepusher.xacro (robot description, xacro)
@@ -10,4 +10,7 @@
         <color rgba="0 0 0 1" />
     </material>
+    <material name="red">
+        <color rgba="1 0 0 1" />
+    </material>
     <material name="blue">
         <color rgba="0.2 0.2 1 1" />

File: description/robot.urdf.xacro (robot description, xacro)
@@ -2,7 +2,8 @@
 <robot xmlns:xacro="http://www.ros.org/wiki/xacro"  name="pulsepusher">
     <xacro:include filename="pulsepusher.xacro" />
+    <xacro:include filename="turret.xacro"/>
+    <xacro:include filename="camera.xacro" />
     <xacro:include filename="gazebo_control.xacro"/>
  <!--    <xacro:include filename="lidar.xacro" />
-    <xacro:include filename="camera.xacro" />
      <xacro:include filename="ros2_control.xacro" /> -->
 <!--
